File: rc2014-82c55-ide.kicad_pcb (KiCad board)
At the start: 2 copper layers, 100 x 50 mm, 13 parts, among them J1 CONN_02X06, J2 IDE connector, P1 RC2014 BUS, U1 82C55A_PLCC, U2 74HCT688, U3 74HCT04

Commit message: WIP
Parts:
- removed R2: 10K, Resistors_THT:R_Axial_DIN0207_L6.3mm_D2.5mm_P7.62mm_Horizontal
- added J3: IDE connector, Pin_Headers:Pin_Header_Straight_2x22_Pitch2.00mm, F.Cu at (93.7, 127.0)
- moved R1 27.9 mm to (149.9, 123.8), turned to 180 degrees
- moved C2 22.2 mm to (98.4, 156.2), turned to 180 degrees
- moved U3 17.2 mm to (139.7, 151.1)
- moved U2 16.0 mm to (76.2, 150.5), turned to 90 degrees
- moved C3 15.3 mm to (139.1, 137.8)
- moved C1 14.5 mm to (76.2, 137.8)
- moved U1 6.48 mm to (115.6, 146.7), turned to 180 degrees
- moved J1 2.01 mm to (62.2, 136.5)
- moved RN1 2.01 mm to (70.5, 156.8)
- moved D1 1.27 mm to (149.9, 118.1)
Connections:
- J2 pad 33: /DA0 -> /DA1
- J2 pad 35: /DA1 -> /DA0
- U1 pad 39: //RESET -> /RESET
- U3 pad 3: /INTRQ -> //RESET
- U3 pad 4: (no net) -> /RESET
Routing:
- net GND: track 41.5 -> 167.7 mm, vias 0 -> 1
- net //DRESET: track 0.00 -> 75.1 mm, vias 0 -> 1
- net VCC: track 0.00 -> 53.7 mm
- net //PIO_CS: track 0.00 -> 51.8 mm
- net /PB7: track 0.00 -> 47.1 mm
- net /PC1: track 0.00 -> 45.9 mm
- net /D7: track 0.00 -> 43.8 mm
- net /A7: track 55.9 -> 14.2 mm
- net /PB5: track 0.00 -> 41.1 mm
- net //DCS0: track 17.9 -> 57.4 mm, vias 0 -> 1
- net /PB6: track 0.00 -> 38.3 mm
- net /PB3: track 0.00 -> 37.6 mm
- net /PB4: track 0.00 -> 36.3 mm
- net /A1: track 0.00 -> 36.1 mm
- net /PC3: track 0.00 -> 35.7 mm, vias 0 -> 1
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Other:
- net class Default: clearance 0.254 -> 0.127; via_dia 0.6858 -> 0.508; via_drill 0.3302 -> 0.254
- net class gnd removed
- net class vcc removed
- rule trace_clearance: 0.254 -> 0.127
- rule via_min_drill: 0.3302 -> 0.254
- rule via_min_size: 0.6858 -> 0.508

Commit message: Relayout
Parts:
- added SW1: SW_DIP_x06, Buttons_Switches_THT:SW_DIP_x6_W7.62mm_Slide, F.Cu at (82.5, 128.9)
- C1, C2, C3: footprint Capacitors_THT:C_Disc_D3.8mm_W2.6mm_P2.50mm -> Capacitors_THT:C_Disc_D3.0mm_W2.0mm_P2.50mm
- J1: value CONN_02X06 -> CONN_02X13; footprint Pin_Headers:Pin_Header_Straight_2x06_Pitch2.54mm -> Pin_Headers:Pin_Header_Straight_2x13_Pitch2.54mm
- J2: footprint Pin_Headers:Pin_Header_Angled_2x20_Pitch2.54mm -> Pin_Headers:Pin_Header_Straight_2x20_Pitch2.54mm
- moved J1 94.5 mm to (156.2, 127.0)
- moved C3 45.7 mm to (94.6, 148.6), turned to 90 degrees
- moved U3 41.5 mm to (98.4, 154.9)
- moved C2 21.8 mm to (120.0, 153.1), turned to 270 degrees
- moved U1 19.1 mm to (134.6, 144.8)
- moved C1 17.2 mm to (62.9, 148.6), turned to 90 degrees
- moved RN1 14.7 mm to (69.2, 142.2), turned to 0 degrees
- moved U2 10.5 mm to (66.7, 154.9)
- moved R1 1.90 mm to (151.8, 123.8)
- moved J3 0.75 mm to (93.5, 127.7)
- moved J2 0.63 mm to (90.8, 119.4)
Connections:
- J1 pad 1: GND -> /DA0
- J1 pad 10: Net-(J1-Pad10) -> /PA4
- J1 pad 11: GND -> /PC5
- J1 pad 12: Net-(J1-Pad12) -> /PA5
- J1 pad 2: Net-(J1-Pad2) -> /PA0
- J1 pad 3: GND -> /DA1
- J1 pad 4: Net-(J1-Pad4) -> /PA1
- J1 pad 5: GND -> /DA2
- J1 pad 6: Net-(J1-Pad6) -> /PA2
- J1 pad 7: GND -> /PC3
- J1 pad 8: Net-(J1-Pad8) -> /PA3
- J1 pad 9: GND -> /PC4
- J2 pad 31: /INTRQ -> (no net)
- J3 pad 31: /INTRQ -> (no net)
- RN1 pad 1: VCC -> GND
- RN1 pad 4: Net-(J1-Pad12) -> Net-(RN1-Pad4)
- RN1 pad 5: Net-(J1-Pad10) -> Net-(RN1-Pad5)
- RN1 pad 6: Net-(J1-Pad8) -> Net-(RN1-Pad6)
- RN1 pad 7: Net-(J1-Pad6) -> Net-(RN1-Pad7)
- RN1 pad 8: Net-(J1-Pad4) -> Net-(RN1-Pad8)
- RN1 pad 9: Net-(J1-Pad2) -> Net-(RN1-Pad9)
- U1 pad 13: /DA2 -> /PC6
- U1 pad 15: /DA1 -> /PC4
- U1 pad 16: /PC0 -> /DA0
- U1 pad 17: /PC1 -> /DA1
- U1 pad 18: /DA0 -> /DA2
- U2 pad 12: Net-(J1-Pad10) -> Net-(RN1-Pad5)
- U2 pad 14: Net-(J1-Pad12) -> Net-(RN1-Pad4)
- U2 pad 3: Net-(J1-Pad2) -> Net-(RN1-Pad9)
- U2 pad 5: Net-(J1-Pad4) -> Net-(RN1-Pad8)
- U2 pad 7: Net-(J1-Pad6) -> Net-(RN1-Pad7)
- U2 pad 9: Net-(J1-Pad8) -> Net-(RN1-Pad6)
- U3 pad 11: /PC1 -> /PC6
- U3 pad 5: /PC0 -> /PC5
- U3 pad 9: /PC5 -> /PC4
Routing:
- net VCC: track 53.7 -> 143.1 mm
- net /PA6: track 9.76 -> 81.7 mm, vias 0 -> 1
- net /PC6: track 0.00 -> 68.4 mm, vias 0 -> 2
- net /PA7: track 9.99 -> 71.0 mm, vias 0 -> 1
- net /PB2: track 34.9 -> 81.9 mm, vias 0 -> 1
- net /PB3: track 37.6 -> 84.0 mm, vias 0 -> 1
- net /PC1: track 45.9 -> 0.00 mm
- net /DA0: track 10.9 -> 56.3 mm
- net Net-(J1-Pad8): track 45.4 -> 0.00 mm
- net /PC0: track 43.2 -> 0.00 mm, vias 1 -> 0
- net /PB6: track 38.3 -> 81.2 mm, vias 0 -> 2
- net /PA1: track 35.3 -> 76.0 mm, vias 0 -> 1
- net Net-(J1-Pad2): track 38.9 -> 0.00 mm
- net GND: track 167.7 -> 206.5 mm, vias 1 -> 0
- net Net-(J1-Pad6): track 38.6 -> 0.00 mm
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
Commit message: WIP
Parts:
- added J5: CONN_01X03, Pin_Headers:Pin_Header_Straight_1x03_Pitch2.54mm, F.Cu at (156.8, 136.5)
- added REF***: OSHW-Logo2_14.6x12mm_SilkScreen, Symbols:OSHW-Logo2_14.6x12mm_SilkScreen, F.Cu at (79.4, 121.3)
- D1: footprint LEDs:LED_D3.0mm_Horizontal_O3.81mm_Z6.0mm -> LEDs:LED_D1.8mm_W3.3mm_H2.4mm
- J1: value CONN_02X13 -> CONN_01X02; footprint Pin_Headers:Pin_Header_Straight_2x13_Pitch2.54mm -> Connectors:PINHEAD1-2
- moved J1 9.44 mm to (149.2, 133.3)
- moved D1 1.91 mm to (148.0, 118.1), turned to 0 degrees
Connections:
- J1 pad 1: /DA0 -> /EXT_VCC
- J1 pad 2: /PA0 -> GND
- J3 pad 41: VCC -> /IDE_VCC
- J3 pad 42: VCC -> /IDE_VCC
Routing:
- net GND: track 206.5 -> 291.4 mm
- net VCC: track 143.1 -> 186.3 mm, vias 0 -> 2
- net /PB3: track 84.0 -> 46.1 mm
- net /PB2: track 81.9 -> 45.1 mm
- net /PB6: track 81.2 -> 45.5 mm, vias 2 -> 1
- net //M1: track 0.00 -> 35.6 mm, vias 0 -> 3
- net /DA0: track 56.3 -> 23.9 mm
- net /IDE_VCC: track 0.00 -> 31.2 mm
- net /DA1: track 50.7 -> 20.1 mm, vias 1 -> 0
- net /PC6: track 68.4 -> 40.4 mm, vias 2 -> 1
- net /PC5: track 60.5 -> 32.7 mm, vias 3 -> 0
- net /PA0: track 73.1 -> 48.4 mm, vias 2 -> 0
- net /PA5: track 81.5 -> 59.1 mm
- net Net-(RN1-Pad8): track 9.35 -> 31.3 mm
- net /PA1: track 76.0 -> 55.2 mm
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- added copper zone on F.Cu, net GND
Other:
- net class Default: via_dia 0.508 -> 0.6; via_drill 0.254 -> 0.3
- rule via_min_drill: 0.254 -> 0.3
- rule via_min_size: 0.508 -> 0.6
- board text added: "2017 Ed Brindley"
- board text added: "RC2014 IDE Adapter"
- board text added: "Rev 1"
- board text added: "github.com/electrified/rc2014-82c55-ide"
- board text removed: "github.com/electrified/rc2014-ym2149"

Commit message: WIP
Parts:
- removed REF***: OSHW-Logo2_14.6x12mm_SilkScreen, Symbols:OSHW-Logo2_14.6x12mm_SilkScreen
- added JP1: Jumper_Dual, Pin_Headers:Pin_Header_Straight_1x03_Pitch2.54mm, F.Cu at (101.7, 140.1)
- added JP2: Jumper_Dual, Pin_Headers:Pin_Header_Straight_1x03_Pitch2.54mm, F.Cu at (98.5, 140.1)
- added JP3: Jumper_Dual, Pin_Headers:Pin_Header_Straight_1x03_Pitch2.54mm, F.Cu at (95.3, 140.1)
- added JP4: Jumper_Dual, Pin_Headers:Pin_Header_Straight_1x03_Pitch2.54mm, F.Cu at (92.2, 140.1)
- RN1: footprint Resistors_THT:R_Array_SIP9 -> Resistors_THT:R_Array_SIP8
- moved J5 16.5 mm to (152.4, 152.4)
- moved J1 4.26 mm to (151.1, 137.2)
- moved RN1 2.54 mm to (66.7, 142.2)
- moved SW1 2.01 mm to (80.6, 129.5)
Connections:
- SW1 pad 10: Net-(RN1-Pad7) -> Net-(RN1-Pad6)
- SW1 pad 11: Net-(RN1-Pad8) -> Net-(RN1-Pad7)
- SW1 pad 12: Net-(RN1-Pad9) -> Net-(RN1-Pad8)
- SW1 pad 7: Net-(RN1-Pad4) -> Net-(RN1-Pad3)
- SW1 pad 8: Net-(RN1-Pad5) -> Net-(RN1-Pad4)
- SW1 pad 9: Net-(RN1-Pad6) -> Net-(RN1-Pad5)
- U1 pad 16: /DA0 -> /PC0
- U1 pad 17: /DA1 -> /PC1
- U2 pad 12: Net-(RN1-Pad5) -> Net-(RN1-Pad4)
- U2 pad 14: Net-(RN1-Pad4) -> Net-(RN1-Pad3)
- U2 pad 16: Net-(RN1-Pad3) -> VCC
- U2 pad 3: Net-(RN1-Pad9) -> Net-(RN1-Pad8)
- U2 pad 5: Net-(RN1-Pad8) -> Net-(RN1-Pad7)
- U2 pad 7: Net-(RN1-Pad7) -> Net-(RN1-Pad6)
- U2 pad 9: Net-(RN1-Pad6) -> Net-(RN1-Pad5)
- U3 pad 11: /PC6 -> /DIOR
- U3 pad 9: /PC4 -> /DCS1
Routing:
- net /PC1: track 0.00 -> 43.7 mm, vias 0 -> 1
- net /PC0: track 0.00 -> 40.5 mm, vias 0 -> 1
- net Net-(RN1-Pad9): track 35.2 -> 0.00 mm
- net VCC: track 186.3 -> 214.6 mm, vias 2 -> 3
- net /DA1: track 20.1 -> 46.6 mm, vias 0 -> 1
- net /DIOR: track 0.00 -> 22.2 mm
- net /DCS1: track 0.00 -> 20.9 mm
- net /DA0: track 23.9 -> 41.2 mm, vias 0 -> 1
- net Net-(RN1-Pad3): track 6.13 -> 19.6 mm
- net /PC4: track 26.4 -> 39.7 mm, vias 0 -> 1
- net Net-(RN1-Pad5): track 19.3 -> 29.3 mm
- net /PC6: track 40.4 -> 50.4 mm
- net Net-(RN1-Pad6): track 29.2 -> 20.8 mm
- net //PIO_CS: track 90.1 -> 83.1 mm, vias 1 -> 4
- net Net-(RN1-Pad4): track 16.5 -> 22.1 mm
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
Commit message: reroute
Parts:
- added REF***: OSHW-Logo2_14.6x12mm_SilkScreen, Symbols:OSHW-Logo2_14.6x12mm_SilkScreen, B.Cu at (78.7, 121.9)
- moved JP1 10.1 mm to (111.8, 141.0)
- moved JP2 9.47 mm to (108.0, 141.0)
- moved JP3 8.84 mm to (104.1, 141.0)
- moved JP4 8.21 mm to (100.3, 141.0)
- moved J2 2.62 mm to (90.2, 121.9)
- moved C1 2.54 mm to (62.9, 151.1)
- moved C3 2.54 mm to (94.6, 151.1)
- moved R1 1.27 mm to (153.0, 123.8)
- moved U1 1.27 mm to (134.6, 146.1)
- moved U2 1.27 mm to (66.7, 156.2)
- moved U3 1.27 mm to (98.4, 156.2)
- moved C2 1.23 mm to (120.0, 154.3)
- moved J3 1.18 mm to (93.3, 128.9)
- moved RN1 0.63 mm to (66.7, 142.9)
Routing:
- net /PA7: track 65.6 -> 115.5 mm, vias 1 -> 0
- net GND: track 289.7 -> 241.5 mm
- net /PA4: track 59.3 -> 92.9 mm, vias 1 -> 0
- net /PA1: track 51.0 -> 81.3 mm, vias 1 -> 0
- net VCC: track 214.6 -> 184.5 mm, vias 3 -> 0
- net //DIOW: track 41.1 -> 58.5 mm, vias 1 -> 0
- net Net-(RN1-Pad6): track 20.8 -> 36.7 mm
- net /PC0: track 40.5 -> 27.3 mm, vias 1 -> 0
- net /PC6: track 50.4 -> 37.5 mm, vias 1 -> 0
- net /PC1: track 43.7 -> 32.4 mm, vias 1 -> 0
- net //DRESET: track 42.9 -> 32.2 mm
- net /PB2: track 45.1 -> 55.6 mm, vias 1 -> 0
- net /DA1: track 46.6 -> 36.6 mm
- net /A1: track 59.1 -> 68.9 mm, vias 0 -> 1
- net Net-(RN1-Pad5): track 29.3 -> 39.0 mm
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- added copper zone on B.Cu, net GND
- removed copper zone on F.Cu, net GND
Other:
- net class Power added: clearance 0.127, trace_width 0.635, via_dia 0.6, via_drill 0.3
- board text added: "1-2 2-3 JP1: DA0 PC0 PC4 JP2: DCS1 PC4 PC0 JP3: DA1 PC1 PC6 JP4: DIOR PC6 PC1"
- board text added: "5v"
- board text added: "A2 A3 A4 A5 A6 A7"
- board text added: "Activity"
- board text added: "Bus"
- board text added: "Default ["
- board text added: "Ext"
- board text added: "GND"
- board text added: "VCC"

Commit message: R1 as submitted to allpcb
Parts:
- added R2: 10K, Resistors_THT:R_Axial_DIN0207_L6.3mm_D2.5mm_P7.62mm_Horizontal, F.Cu at (88.3, 134.0)
- added R3: 10K, Resistors_THT:R_Axial_DIN0207_L6.3mm_D2.5mm_P7.62mm_Horizontal, F.Cu at (88.3, 137.8)
- added R4: 10K, Resistors_THT:R_Axial_DIN0207_L6.3mm_D2.5mm_P7.62mm_Horizontal, F.Cu at (88.3, 141.6)
Connections:
- J2 pad 21: (no net) -> /DMARQ
- J2 pad 28: (no net) -> GND
- J2 pad 29: (no net) -> /DMACK
- J3 pad 21: (no net) -> /DMARQ
- J3 pad 28: (no net) -> GND
- J3 pad 29: (no net) -> /DMACK
Routing:
- net VCC: track 184.5 -> 247.4 mm
- net /PA7: track 115.5 -> 67.5 mm
- net /DMACK: track 0.00 -> 41.2 mm, vias 0 -> 1
- net /PA4: track 92.9 -> 61.2 mm
- net /PA1: track 81.3 -> 51.1 mm
- net /DMARQ: track 0.00 -> 29.0 mm
- net /PB2: track 55.6 -> 80.5 mm
- net /PB6: track 43.4 -> 65.8 mm, vias 0 -> 1
- net //DIOW: track 58.5 -> 37.4 mm, vias 0 -> 2
- net /PB5: track 43.1 -> 62.2 mm
- net GND: track 241.5 -> 224.8 mm
- net /PB0: track 48.4 -> 63.8 mm, vias 1 -> 0
- net Net-(RN1-Pad6): track 36.7 -> 21.7 mm
- net /PB7: track 45.6 -> 58.3 mm, vias 0 -> 1
- net /A1: track 68.9 -> 56.7 mm
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Other:
- board text added: "] Default"
- board text removed: "Default ["
