File: rc2014-82c55-ide.kicad_sch (KiCad schematic)
At the start: 22 parts, among them J1 Conn_01x02, J2 Conn_02x20_Odd_Even, J3 Conn_02x22_Odd_Even, J5 Conn_01x02, P1 Conn_01x39, SW1 SW_DIP_x06, U1 82C55A_PLCC, U2 74HCT688, U3 74HCT04

Commit message: Further kicad 6 migration
Parts:
- added unit 7 of U3
- C1, C2, C3: footprint Capacitors_THT:C_Disc_D3.0mm_W2.0mm_P2.50mm -> Capacitor_THT:C_Disc_D3.0mm_W2.0mm_P2.50mm
- D1: footprint LEDs:LED_D3.0mm -> LED_THT:LED_D3.0mm
- J1: footprint Connectors:PINHEAD1-2 -> Connector_PinHeader_2.54mm:PinHeader_1x02_P2.54mm_Vertical
- J2: footprint Pin_Headers:Pin_Header_Straight_2x20_Pitch2.54mm -> Connector_PinHeader_2.54mm:PinHeader_2x20_P2.54mm_Vertical
- J3: footprint Pin_Headers:Pin_Header_Straight_2x22_Pitch2.00mm -> Connector_PinHeader_2.00mm:PinHeader_2x22_P2.00mm_Vertical
- J5: footprint Pin_Headers:Pin_Header_Straight_1x02_Pitch2.54mm -> Connector_PinHeader_2.54mm:PinHeader_1x02_P2.54mm_Vertical
- JP1, JP2, JP3, JP4: footprint Pin_Headers:Pin_Header_Straight_1x03_Pitch2.54mm -> Connector_PinHeader_2.54mm:PinHeader_1x03_P2.54mm_Vertical
- R1, R2, R3, R4: footprint Resistors_THT:R_Axial_DIN0207_L6.3mm_D2.5mm_P7.62mm_Horizontal -> Resistor_THT:R_Axial_DIN0207_L6.3mm_D2.5mm_P7.62mm_Horizontal
- SW1: footprint Buttons_Switches_THT:SW_DIP_x6_W7.62mm_Slide -> Button_Switch_THT:SW_DIP_SPSTx06_Slide_9.78x17.42mm_W7.62mm_P2.54mm
- U2: footprint Housings_DIP:DIP-20_W7.62mm_Socket_LongPads -> Package_DIP:DIP-20_W7.62mm_Socket_LongPads
- U3: footprint Housings_DIP:DIP-14_W7.62mm_Socket_LongPads -> Package_DIP:DIP-14_W7.62mm_Socket_LongPads
Connections:
- net GND: now also U3.7 (GND)
- net VCC: now also U3.14 (VCC)
- net /ACT renamed ~{ACT}
- net /DCS0 renamed ~{DCS0}
- net /DCS1 renamed ~{DCS1}
- net /DIOR renamed ~{DIOR}
- net /DIOW renamed ~{DIOW}
- net /DRESET renamed ~{DRESET}
- net /IORQ renamed ~{IORQ}
- net /M1 renamed ~{M1}
- net /PIO_CS renamed ~{PIO_CS}
- net /RD renamed ~{RD}
- net /RESET renamed ~{RESET}
- net /WR renamed ~{WR}
Other:
- note added: "CSEL"
- moved on the sheet: J2, J3
